File: board/spacelock.kicad_pcb (KiCad board)
At the start: 2 copper layers, 2 parts, among them J1 CP-036AHPJ, U1 SFTPOWER-V1

Commit message: board: main connectivity
Parts:
- added A1: Pololu_Breakout_DRV8825, Module:Pololu_Breakout-16_15.2x20.3mm, F.Cu at (67.3, 79.0)
- added C1: 10uF 6.3V, Capacitor_SMD:C_1206_3216Metric_Pad1.42x1.75mm_HandSolder, F.Cu at (164.9, 67.3)
- added C10: 4.7uF, Capacitor_SMD:C_0603_1608Metric_Pad1.05x0.95mm_HandSolder, F.Cu at (90.6, 111.8)
- added C11: 100nF, Capacitor_SMD:C_0603_1608Metric_Pad1.05x0.95mm_HandSolder, F.Cu at (89.3, 106.7)
- added C12: 100nF, Capacitor_SMD:C_0603_1608Metric_Pad1.05x0.95mm_HandSolder, F.Cu at (90.6, 102.9)
- added C13: 100nF, Capacitor_SMD:C_0603_1608Metric_Pad1.05x0.95mm_HandSolder, F.Cu at (97.8, 101.6)
- added C2: 100nF, Capacitor_SMD:C_0603_1608Metric_Pad1.05x0.95mm_HandSolder, F.Cu at (76.2, 161.7)
- added C3: 22 uF 25V, Capacitor_SMD:C_1206_3216Metric_Pad1.42x1.75mm_HandSolder, F.Cu at (187.2, 84.1)
- added C4: 100nF, Capacitor_SMD:C_0603_1608Metric_Pad1.05x0.95mm_HandSolder, F.Cu at (84.2, 158.8)
- added C5: 18pF, Capacitor_SMD:C_0603_1608Metric_Pad1.05x0.95mm_HandSolder, F.Cu at (104.1, 138.4)
- added C6: 18pF, Capacitor_SMD:C_0603_1608Metric_Pad1.05x0.95mm_HandSolder, F.Cu at (109.2, 137.6)
- added C7: 100nF, Capacitor_SMD:C_0603_1608Metric_Pad1.05x0.95mm_HandSolder, F.Cu at (93.6, 132.1)
- added C8: 4.7uF, Capacitor_SMD:C_0603_1608Metric_Pad1.05x0.95mm_HandSolder, F.Cu at (91.8, 121.9)
- added C9: 100nF, Capacitor_SMD:C_0603_1608Metric_Pad1.05x0.95mm_HandSolder, F.Cu at (91.0, 116.8)
- added D1: ZMM5248_R1_00001 18V, Diode_SMD:D_MiniMELF_Handsoldering, F.Cu at (197.4, 83.1)
- added D2: LED2, LED_SMD:LED_0805_2012Metric_Pad1.15x1.40mm_HandSolder, F.Cu at (124.2, 111.2)
- added D3: LED1, LED_SMD:LED_0805_2012Metric_Pad1.15x1.40mm_HandSolder, F.Cu at (123.9, 116.6)
- added D4: LED_PWR, LED_SMD:LED_0805_2012Metric_Pad1.15x1.40mm_HandSolder, F.Cu at (123.7, 151.4)
- added D5: LED0, LED_SMD:LED_0805_2012Metric_Pad1.15x1.40mm_HandSolder, F.Cu at (123.9, 122.6)
- added D6: LED_TIMESTATE, LED_SMD:LED_0805_2012Metric_Pad1.15x1.40mm_HandSolder, F.Cu at (123.9, 144.5)
- added D7: LED_TIMETICK, LED_SMD:LED_0805_2012Metric_Pad1.15x1.40mm_HandSolder, F.Cu at (123.9, 138.2)
- added D8: LED_DOORSTATE, LED_SMD:LED_0805_2012Metric_Pad1.15x1.40mm_HandSolder, F.Cu at (124.2, 132.0)
- added J2: Raspberry_Pi_Zero_W, Module:Raspberry_Pi_Zero_Socketed_THT_FaceDown_MountingHoles, F.Cu at (115.1, 45.7)
- added J3: USB_B_Micro, sft:Amphenol_10118194, F.Cu at (27.9, 110.8)
- added M1: Stepper_Motor_bipolar, Connector_PinHeader_2.54mm:PinHeader_1x04_P2.54mm_Horizontal, F.Cu at (35.8, 79.5)
- added R1: 4k7, Resistor_SMD:R_0603_1608Metric_Pad1.05x0.95mm_HandSolder, F.Cu at (87.6, 171.4)
- added R10: 4k7, Resistor_SMD:R_0603_1608Metric_Pad1.05x0.95mm_HandSolder, F.Cu at (131.8, 151.4)
- added R11: 4k7, Resistor_SMD:R_0603_1608Metric_Pad1.05x0.95mm_HandSolder, F.Cu at (40.3, 103.6)
- added R12: 22, Resistor_SMD:R_0603_1608Metric_Pad1.05x0.95mm_HandSolder, F.Cu at (55.9, 99.1)
- added R13: 22, Resistor_SMD:R_0603_1608Metric_Pad1.05x0.95mm_HandSolder, F.Cu at (55.9, 102.9)
- added R2: 4k7, Resistor_SMD:R_0603_1608Metric_Pad1.05x0.95mm_HandSolder, F.Cu at (94.0, 171.8)
- added R3: 1k, Resistor_SMD:R_0603_1608Metric_Pad1.05x0.95mm_HandSolder, F.Cu at (130.7, 111.1)
- added R4: 3k3, Resistor_SMD:R_0603_1608Metric_Pad1.05x0.95mm_HandSolder, F.Cu at (131.3, 115.7)
- added R5: 1k, Resistor_SMD:R_0603_1608Metric_Pad1.05x0.95mm_HandSolder, F.Cu at (131.3, 121.3)
- added R6: 1k, Resistor_SMD:R_0603_1608Metric_Pad1.05x0.95mm_HandSolder, F.Cu at (131.7, 144.5)
- added R7: 3k3, Resistor_SMD:R_0603_1608Metric_Pad1.05x0.95mm_HandSolder, F.Cu at (131.7, 138.2)
- added R8: 1k, Resistor_SMD:R_0603_1608Metric_Pad1.05x0.95mm_HandSolder, F.Cu at (131.6, 131.2)
- added R9: 10k, Resistor_SMD:R_0603_1608Metric_Pad1.05x0.95mm_HandSolder, F.Cu at (134.7, 98.3)
- added SW1: RESET, Button_Switch_THT:SW_PUSH_6mm_H4.3mm, F.Cu at (88.9, 144.8)
- added SW2: FORCE_DFU, Button_Switch_THT:SW_PUSH_6mm_H4.3mm, F.Cu at (119.9, 97.0)
- added U2: DCF1-Pollin, sft:DCF1-Pollin, F.Cu at (167.6, 62.2)
- added U3: TLV76033, Package_TO_SOT_SMD:SOT-23, F.Cu at (77.2, 152.4)
- added U4: STM32F103C8Tx, Package_QFP:LQFP-48_7x7mm_P0.5mm, F.Cu at (99.5, 91.2)
- added U5: USBLC6-4SC6, Package_TO_SOT_SMD:SOT-23-6, F.Cu at (40.4, 108.0)
- added X1: OLED_I2C_128x64, sft:OLED_128x64_096in_IZOKEE, F.Cu at (73.7, 179.1)
- added X2: SFT_DEBUG_CONNECTOR-DUT, Connector:Tag-Connect_TC2050-IDC-FP_2x05_P1.27mm_Vertical, F.Cu at (117.3, 82.3)
- added Y1: 8.000 MHz, Crystal:Crystal_HC49-U_Vertical, F.Cu at (109.2, 132.1)
- moved J1 63.1 mm to (37.6, 91.2), turned to 270 degrees
- moved U1 46.2 mm to (71.1, 111.8)
