File: board/spacelock.sch (KiCad schematic (older format))
At the start: 11 parts, among them J1 CP-036AHPJ, U1 SFTPOWER-V1

Commit message: board: main connectivity
Parts:
- added C10, C8: 4.7uF, Capacitor_SMD:C_0603_1608Metric_Pad1.05x0.95mm_HandSolder, symbol Device:C
- added C11, C12, C13, C7, C9: 100nF, Capacitor_SMD:C_0603_1608Metric_Pad1.05x0.95mm_HandSolder, symbol Device:C
- added C5, C6: 18pF, Capacitor_SMD:C_0603_1608Metric_Pad1.05x0.95mm_HandSolder, symbol Device:C
- added D2: LED2, LED_SMD:LED_0805_2012Metric_Pad1.15x1.40mm_HandSolder, symbol Device:LED
- added D3: LED1, LED_SMD:LED_0805_2012Metric_Pad1.15x1.40mm_HandSolder, symbol Device:LED
- added D4: LED_PWR, LED_SMD:LED_0805_2012Metric_Pad1.15x1.40mm_HandSolder, symbol Device:LED
- added D5: LED0, LED_SMD:LED_0805_2012Metric_Pad1.15x1.40mm_HandSolder, symbol Device:LED
- added D6: LED_TIMESTATE, LED_SMD:LED_0805_2012Metric_Pad1.15x1.40mm_HandSolder, symbol Device:LED
- added D7: LED_TIMETICK, LED_SMD:LED_0805_2012Metric_Pad1.15x1.40mm_HandSolder, symbol Device:LED
- added D8: LED_DOORSTATE, LED_SMD:LED_0805_2012Metric_Pad1.15x1.40mm_HandSolder, symbol Device:LED
- added J2: Raspberry_Pi_Zero_W, Module:Raspberry_Pi_Zero_Socketed_THT_FaceDown_MountingHoles, symbol sft:Raspberry_Pi_Zero_W
- added J3: USB_B_Micro, sft:Amphenol_10118194, symbol Connector:USB_B_Micro
- added J?: External Extension, symbol Connector_Generic:Conn_02x04_Odd_Even
- added R1, R10, R11, R2: 4k7, Resistor_SMD:R_0603_1608Metric_Pad1.05x0.95mm_HandSolder, symbol Device:R
- added R12, R13: 22, Resistor_SMD:R_0603_1608Metric_Pad1.05x0.95mm_HandSolder, symbol Device:R
- added R3, R5, R6, R8: 1k, Resistor_SMD:R_0603_1608Metric_Pad1.05x0.95mm_HandSolder, symbol Device:R
- added R4, R7: 3k3, Resistor_SMD:R_0603_1608Metric_Pad1.05x0.95mm_HandSolder, symbol Device:R
- added R9: 10k, Resistor_SMD:R_0603_1608Metric_Pad1.05x0.95mm_HandSolder, symbol Device:R
- added SW1: RESET, Button_Switch_THT:SW_PUSH_6mm_H4.3mm, symbol Switch:SW_Push
- added SW2: FORCE_DFU, Button_Switch_THT:SW_PUSH_6mm_H4.3mm, symbol Switch:SW_Push
- added SW? (x2): SW_Push, symbol Switch:SW_Push
- added SW?: Rotary_Encoder, sft:Bourns_PEC16_2xxxF, symbol Device:Rotary_Encoder
- added U4: STM32F103C8Tx, Package_QFP:LQFP-48_7x7mm_P0.5mm, symbol MCU_ST_STM32F1:STM32F103C8Tx
- added U5: USBLC6-4SC6, Package_TO_SOT_SMD:SOT-23-6, symbol sft:USBLC6-4SC6
- added U? (x2): 74AHC1G08, symbol 74xGxx:74AHC1G08
- added X1: OLED_I2C_128x64, sft:OLED_128x64_096in_IZOKEE, symbol sft:OLED_I2C_128x64
- added X2: SFT_DEBUG_CONNECTOR-DUT, Connector:Tag-Connect_TC2050-IDC-FP_2x05_P1.27mm_Vertical, symbol sft:SFT_DEBUG_CONNECTOR-DUT
- added Y1: 8.000 MHz, Crystal:Crystal_HC49-U_Vertical, symbol Device:Crystal
- D1: renamed from D?; MPN (none) -> ZMM5248B
- M1: renamed from M?; footprint (none) -> Connector_PinHeader_2.54mm:PinHeader_1x04_P2.54mm_Horizontal; MPN (none) -> Molex 74099-0004
- U3: renamed from U?; footprint (none) -> Package_TO_SOT_SMD:SOT-23
- gave numbers to parts that had none: 6
Connections:
- net +12V: now also X2.10 (V_SUPPLY)
- net +3V3: now also C10.1, C11.1, C12.1, C13.1, C8.1, C9.1, R1.2, R10.1, R2.2, R9.1, SW?.2, SW?.2, U4.1 (VBAT), U4.24 (VDD), U4.36 (VDD), U4.48 (VDD), U4.9 (VDDA), X2.9 (V_FB)
- net +5V: now also A1.13 (~RST), J2.2 (5V), J2.4 (5V), J3.1 (VBUS), J?.1 (Pin_1), R11.1, U5.5, X1.2 (VCC)
- net GND: now also C10.2, C11.2, C12.2, C13.2, C5.2, C6.2, C7.2, C8.2, C9.2, D2.1 (K), D3.1 (K), D4.1 (K), D5.1 (K), D6.1 (K), D7.1 (K), D8.1 (K), J2.14 (GND), J2.20 (GND), J2.25 (GND), J2.30 (GND), J2.34 (GND), J2.39 (GND), J2.6 (GND), J2.9 (GND), J3.4 (ID), J3.5 (GND), J3.6 (Shield), J?.2 (Pin_2), SW1.1, SW2.1, U4.44 (BOOT0), U5.2, U?.3 (GND), U?.3 (GND), X1.1 (GND), X2.1 (GND)
- net TIME_SIGNAL: now also R7.2, U4.29 (PA8), X2.7 (AUX)
- net MOT_MODE0: now reaches A1.10 (M0)
- net MOT_MODE0: now also U4.21 (PB10)
- net MOT_MODE1: now reaches A1.11 (M1)
- net MOT_MODE1: now also U4.19 (PB1)
- net MOT_MODE2: now reaches A1.12 (M2)
- net MOT_MODE2: now also U4.18 (PB0)
- net MOT_~SLP: now reaches A1.14 (~SLP)
- net MOT_~SLP: now also U4.16 (PA6)
- net MOT_STEP: now reaches A1.15 (STEP)
- net MOT_STEP: now also U4.15 (PA5)
- net MOT_DIR: now reaches A1.16 (DIR)
- net MOT_DIR: now also U4.14 (PA4)
- new net: C5.1, U4.5 (PD0), Y1.2
- new net: C6.1, U4.6 (PD1), Y1.1
- new net: U?.1, U?.4
- new net: D7.2 (A), R7.1
- new net: D8.2 (A), R8.1
- new net: D6.2 (A), R6.1
- new net: D3.2 (A), R4.2
- new net: D2.2 (A), R3.2
- new net: D5.2 (A), R5.2
- new net: D4.2 (A), R10.2
- new net: J3.2 (D-), R12.1, U5.6
- new net: J3.3 (D+), R13.1, U5.1
- new net CTRL_~RST: C7.1, SW1.2, U4.7 (NRST), X2.2 (RST)
- new net DBG_SWCLK: U4.37 (PA14), X2.3 (SWCLK)
- new net DBG_SWDIO: U4.34 (PA13), X2.8 (SWDIO)
- new net DBG_TRACESWO: U4.39 (PB3), X2.4 (SWO)
- new net DISPLAY_SCL: J?.3 (Pin_3), R1.1, U4.45 (PB8), X1.3 (SCL)
- new net DISPLAY_SDA: J?.4 (Pin_4), R2.1, U4.46 (PB9), X1.4 (SDA)
- new net FORCE_DFU: R9.2, SW2.2, U4.25 (PB12)
- new net LED0: R5.1, U4.10 (PA0)
- new net LED1: R4.1, U4.11 (PA1)
- new net LED2: R3.1, U4.12 (PA2)
- new net LED_DOORSTATE: R8.2, U4.4 (PC15)
- new net LED_TIMESTATE: R6.2, U4.3 (PC14)
- new net MOT_MOVE0: SW?.1, U4.41 (PB5)
- new net MOT_MOVE1: SW?.1, U4.42 (PB6)
- new net PI_RX: J2.10 (GPIO15/RXD), U4.30 (PA9)
- new net PI_TX: J2.8 (GPIO14/TXD), U4.31 (PA10)
- new net USB+: R11.2, R13.2, U4.33 (PA12)
- new net USB-: R12.2, U4.32 (PA11)
- new net VCC: U?.5 (VCC), U?.5 (VCC)
- no-connect marks 0 -> 2
Other:
- note added: "POWER LED"
- note added: "STATUS LEDs"
- note added: "clockwise endstop"
- note added: "counter-clockwise endstop"
- note added: "press during boot to\nforce DFU mode"
- moved on the sheet: C1, C2, C3, C4, D1, U1, U2, U3
