File: board_inside/board_v1/board.kicad_pcb (KiCad board)
At the start: 2 copper layers, 50.9 x 68.3 mm, 101 parts, among them J1 PJ-063AH, J2 Raspberry_Pi_Zero_W, J3 Conn_01x04_Female, J4 Conn_01x06_Female, M1 Stepper_Motor_bipolar, Q1 BC848, SW1 PB, U1 DCF1-Pollin, U10 TLV8811, U2 TPS54302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

Commit message: inner board v1.1, rtc, QR-connector
Parts:
- added BT1: CR3212, Battery:BatteryHolder_Keystone_3000_1x12mm, F.Cu at (122.3, 129.8)
- added C28: 10uF, Capacitor_SMD:C_0603_1608Metric_Pad1.08x0.95mm_HandSolder, F.Cu at (114.8, 110.1)
- added D11: D_Schottky, Diode_SMD:D_SOD-123, F.Cu at (180.8, 86.0)
- added D12: D, Diode_SMD:D_SMB, F.Cu at (180.4, 102.8)
- added F3: Polyfuse_Small, Resistor_SMD:R_1210_3225Metric, F.Cu at (180.3, 110.6)
- added J5: QR_connector, Connector_PinHeader_2.54mm:PinHeader_1x04_P2.54mm_Vertical, F.Cu at (179.7, 119.2)
- added JP5: SolderJumper_2_Open, Jumper:SolderJumper-2_P1.3mm_Open_TrianglePad1.0x1.5mm, F.Cu at (180.2, 96.4)
- added JP6: SolderJumper_2_Open, Jumper:SolderJumper-2_P1.3mm_Open_TrianglePad1.0x1.5mm, F.Cu at (180.2, 92.0)
- added R26: 18k, Resistor_SMD:R_0603_1608Metric_Pad0.98x0.95mm_HandSolder, B.Cu at (146.0, 129.3)
- added R27: 18k, Resistor_SMD:R_0603_1608Metric_Pad0.98x0.95mm_HandSolder, B.Cu at (146.0, 131.0)
- added R28: 1k, Resistor_SMD:R_0603_1608Metric_Pad0.98x0.95mm_HandSolder, F.Cu at (115.6, 107.4)
- added R29: 10k, Resistor_SMD:R_0603_1608Metric_Pad0.98x0.95mm_HandSolder, F.Cu at (119.3, 107.3)
- added R30: 10k, Resistor_SMD:R_0603_1608Metric_Pad0.98x0.95mm_HandSolder, F.Cu at (120.6, 105.7)
- added U9: PCF8523T, Package_SO:SOIC-8_3.9x4.9mm_P1.27mm, F.Cu at (119.6, 112.6)
- added Y2: 32768 Hz, Crystal:Crystal_SMD_EuroQuartz_EQ161-2Pin_3.2x1.5mm_HandSoldering, F.Cu at (116.5, 118.9)
- moved LOGO2 49.3 mm to (116.4, 72.8)
- moved J2 23.8 mm to (106.4, 127.7)
- moved C17 20.8 mm to (122.6, 89.8)
- moved C18 20.8 mm to (128.0, 92.1)
- moved C19 20.8 mm to (129.2, 94.5)
- moved C20 20.8 mm to (126.6, 95.3)
- moved C21 20.8 mm to (126.6, 96.9)
- moved C22 20.8 mm to (126.6, 93.7)
- moved U6 20.8 mm to (127.6, 94.5)
- moved Y1 20.8 mm to (118.0, 96.7)
- moved C11 20.8 mm to (119.8, 92.6)
- moved C12 20.8 mm to (119.8, 96.1)
- moved X2 15.1 mm to (144.9, 94.0)
Connections:
- J2 pad 1: (no net) -> unconnected-(J2-3V3-Pad1)
- J2 pad 11: (no net) -> unconnected-(J2-GPIO17/GEN0-Pad11)
- J2 pad 12: (no net) -> unconnected-(J2-GPIO18/GEN1-Pad12)
- J2 pad 13: (no net) -> unconnected-(J2-GPIO27/GEN2-Pad13)
- J2 pad 15: (no net) -> unconnected-(J2-GPIO22/GEN3-Pad15)
- J2 pad 16: (no net) -> unconnected-(J2-GPIO23/GEN4-Pad16)
- J2 pad 17: (no net) -> unconnected-(J2-3V3-Pad17)
- J2 pad 18: (no net) -> unconnected-(J2-GPIO24/GEN5-Pad18)
- J2 pad 19: (no net) -> unconnected-(J2-MOSI/GPIO10-Pad19)
- J2 pad 21: (no net) -> unconnected-(J2-MISO/GPIO9-Pad21)
- J2 pad 22: (no net) -> unconnected-(J2-GPIO25/GEN6-Pad22)
- J2 pad 23: (no net) -> unconnected-(J2-SCLK/GPIO11-Pad23)
- J2 pad 24: (no net) -> unconnected-(J2-~{CE0}/GPIO8-Pad24)
- J2 pad 26: (no net) -> unconnected-(J2-~{CE1}/GPIO7-Pad26)
- J2 pad 27: (no net) -> unconnected-(J2-ID_SD/GPIO0-Pad27)
- J2 pad 28: (no net) -> unconnected-(J2-ID_SC/GPIO1-Pad28)
- J2 pad 3: (no net) -> unconnected-(J2-SDA/GPIO2-Pad3)
- J2 pad 32: (no net) -> unconnected-(J2-GPIO12-Pad32)
- J2 pad 33: (no net) -> unconnected-(J2-GPIO13-Pad33)
- J2 pad 35: (no net) -> unconnected-(J2-GPIO19-Pad35)
- J2 pad 36: (no net) -> unconnected-(J2-GPIO16-Pad36)
- J2 pad 37: (no net) -> unconnected-(J2-GPIO26-Pad37)
- J2 pad 38: (no net) -> unconnected-(J2-GPIO20-Pad38)
- J2 pad 40: (no net) -> unconnected-(J2-GPIO21-Pad40)
- J2 pad 5: (no net) -> unconnected-(J2-SCL/GPIO3-Pad5)
- J2 pad 7: (no net) -> unconnected-(J2-GCLK/GPIO4-Pad7)
- U3 pad 3: (no net) -> unconnected-(U3-Pad3)
- U3 pad 4: (no net) -> unconnected-(U3-Pad4)
- U6 pad 11: (no net) -> unconnected-(U6-PA1-Pad11)
- U6 pad 12: (no net) -> unconnected-(U6-PA2-Pad12)
- U6 pad 13: (no net) -> /MOT_FAULT
- U6 pad 2: (no net) -> unconnected-(U6-PC13-Pad2)
- U6 pad 20: (no net) -> unconnected-(U6-PB2-Pad20)
- U6 pad 22: (no net) -> unconnected-(U6-PB11-Pad22)
- U6 pad 25: (no net) -> unconnected-(U6-PB12-Pad25)
- U6 pad 26: (no net) -> unconnected-(U6-PB13-Pad26)
- U6 pad 32: (no net) -> unconnected-(U6-PA11-Pad32)
- U6 pad 33: (no net) -> unconnected-(U6-PA12-Pad33)
- U6 pad 38: (no net) -> unconnected-(U6-PA15-Pad38)
- U6 pad 40: (no net) -> unconnected-(U6-PB4-Pad40)
- U6 pad 41: (no net) -> unconnected-(U6-PB5-Pad41)
- U6 pad 42: (no net) -> unconnected-(U6-PB6-Pad42)
- U6 pad 43: (no net) -> unconnected-(U6-PB7-Pad43)
- U6 pad 45: (no net) -> /DISPLAY_SCL
- U6 pad 46: (no net) -> /DISPLAY_SDA
- U7 pad 12: /V3P3 -> Net-(U7-AVREF)
- U7 pad 13: /V3P3 -> Net-(U7-AVREF)
- U7 pad 19: (no net) -> unconnected-(U7-DECAY-Pad19)
- U7 pad 21: (no net) -> unconnected-(U7-~{ENBL}-Pad21)
- U7 pad 23: (no net) -> unconnected-(U7-NC-Pad23)
- U7 pad 27: (no net) -> unconnected-(U7-~{HOME}-Pad27)
Routing:
- net +3V3: track 229.3 -> 304.3 mm, vias 10 -> 17
- net GND: track 583.8 -> 638.5 mm, vias 19 -> 98
- net /CPU_TX: track 98.2 -> 142.8 mm, vias 2 -> 6
- net Net-(BT1-+): track 0.00 -> 41.4 mm
- net /DISPLAY_SCL: track 0.00 -> 40.9 mm
- net /DISPLAY_SDA: track 0.00 -> 39.7 mm
- net +5V: track 156.8 -> 184.5 mm
- net /CTRL_~{RST}: track 61.3 -> 85.3 mm
- net /RPI_CMD: track 45.5 -> 69.3 mm, vias 1 -> 3
- net Net-(D11-K): track 0.00 -> 22.9 mm
- net /TIME_SIGNAL: track 102.6 -> 124.4 mm, vias 4 -> 5
- net /LED_TIMESTATE: track 54.0 -> 73.7 mm
- net /DBG_CMD: track 33.4 -> 52.7 mm, vias 1 -> 3
- net Net-(U7-AVREF): track 0.00 -> 18.5 mm, vias 0 -> 3
- net /CPU_RX: track 29.5 -> 46.8 mm
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Other:
- board size 50.9 x 68.3 mm -> 79.9 x 68.3 mm
- rule solder_mask_min_width: 0.25 -> 0.05
- board text added: "3V3"
- board text added: "5V"
- board text added: "GND"
- board text added: "QR"
- board text added: "Sig"
- board text added: "SpaceLock v1.1"
- board text added: "V+"
- board text removed: "SpaceLock v1"
