File: board_inside/board_v1/board.kicad_sch (KiCad schematic)
At the start: 102 parts, among them J1 PJ-063AH, J2 Raspberry_Pi_Zero_W, J3 Conn_01x04_Female, J4 Conn_01x06_Female, M1 Stepper_Motor_bipolar, Q1 BC848, SW1 PB, U1 DCF1-Pollin, U10 TLV8811, U2 TPS54302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

Commit message: Fix board schematic and documentation after initial commissioning
Other:
- note added: "Measures the combined current of the motor phases. Output MOT_CURRENT = (abs(I(AOUT1)) + abs(I(AOUT2))) * 1V/A. The current is directly proprtional to the torque. Endstop reached if > 600mV >= 20ms"
- note removed: "Measures the combined current of the motor phases. Output MOT_CURRENT = (abs(I(AOUT1)) + abs(I(AOUT2))) * 2V/A. The current is directly proprtional to the torque. Endstop reached if > 600mV >= 20ms"
Changed lines of the file:
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@@
     (stroke (width 0) (type default) (color 0 0 0 0))
   )
-  (text "Measures the combined current of the motor phases.\nOutput MOT_CURRENT = (abs(I(AOUT1)) + abs(I(AOUT2))) * 2V/A.\nThe current is directly proprtional to the torque.\nEndstop reached if > 600mV >= 20ms"
+  (text "Measures the combined current of the motor phases.\nOutput MOT_CURRENT = (abs(I(AOUT1)) + abs(I(AOUT2))) * 1V/A.\nThe current is directly proprtional to the torque.\nEndstop reached if > 600mV >= 20ms"
     (at 203.2 172.72 0)
     (effects (font (size 1.27 1.27)) (justify left bottom))

Commit message: inner board v1.1, rtc, QR-connector
Parts:
- removed LOGO3: Logo, sft:süff_10mm, symbol sft:Logo
- added BT1: CR3212, Battery:BatteryHolder_Keystone_3000_1x12mm, symbol Device:Battery_Cell
- added C28: 10uF, Capacitor_SMD:C_0603_1608Metric_Pad1.08x0.95mm_HandSolder, symbol Device:C
- added D11: D_Schottky, Diode_SMD:D_SOD-123, symbol Device:D_Schottky
- added D12: D, Diode_SMD:D_SMB, symbol Device:D
- added F3: Polyfuse_Small, Resistor_SMD:R_1210_3225Metric, symbol Device:Polyfuse_Small
- added J5: QR_connector, Connector_PinHeader_2.54mm:PinHeader_1x04_P2.54mm_Vertical, symbol Connector_Generic:Conn_01x04
- added JP5, JP6: SolderJumper_2_Open, Jumper:SolderJumper-2_P1.3mm_Open_TrianglePad1.0x1.5mm, symbol Jumper:SolderJumper_2_Open
- added R26, R27: 18k, Resistor_SMD:R_0603_1608Metric_Pad0.98x0.95mm_HandSolder, symbol Device:R
- added R28: 1k, Resistor_SMD:R_0603_1608Metric_Pad0.98x0.95mm_HandSolder, symbol Device:R
- added R29, R30: 10k, Resistor_SMD:R_0603_1608Metric_Pad0.98x0.95mm_HandSolder, symbol Device:R
- added U9: PCF8523T, Package_SO:SOIC-8_3.9x4.9mm_P1.27mm, symbol Timer_RTC:PCF8523T
- added Y2: 32768 Hz, Crystal:Crystal_SMD_EuroQuartz_EQ161-2Pin_3.2x1.5mm_HandSoldering, symbol Device:Crystal
Connections:
- net +3V3: now also JP6.2 (B), R28.1, R29.1, R30.1
- net +5V: now also JP5.2 (B)
- net DISPLAY_SCL: now also R29.2, U9.6 (SCL)
- net DISPLAY_SDA: now also R30.2, U9.5 (SDA)
- net GND: now also BT1.2 (-), C28.2, D11.2 (A), J5.4 (Pin_4), R27.1, U9.4 (VSS)
- net INTERBOARD_BUS_CMD: now also J5.2 (Pin_2)
- net V3P3: now also R26.2; no longer U7.12 (AVREF), U7.13 (BVREF)
- new net: R26.1, R27.2, U7.12 (AVREF), U7.13 (BVREF)
- new net: D11.1 (K), D12.1 (K), F3.1
- new net: F3.2, J5.1 (Pin_1)
- new net: C28.1, R28.2, U9.8 (VDD)
- new net: D12.2 (A), JP5.1 (A), JP6.1 (A)
- new net: U9.1 (OSCI), Y2.2
- new net: U9.2 (OSCO), Y2.1
- new net: BT1.1 (+), U9.3 (VBAT)
Other:
- note added: "RTC"
- note added: "TODO: define ratio!!"
- moved on the sheet: C27, C3, J4, M1, U1
