File: board_inside/board_v1.0/board.kicad_sch (KiCad schematic)
At the start: 116 parts, among them J1 PJ-063AH, J2 Raspberry_Pi_Zero_W, J3 Conn_01x04_Female, J4 Conn_01x06_Female, J5 QR_connector, M1 Stepper_Motor_bipolar, Q1 BC848, SW1 PB, U1 DCF1-Pollin, U10 TLV8811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

Commit message: board v1.1: clean up, create own folder
Parts:
- removed BT1: CR3212, Battery:BatteryHolder_Keystone_3000_1x12mm, symbol Device:Battery_Cell
- removed C28: 10uF, Capacitor_SMD:C_0603_1608Metric_Pad1.08x0.95mm_HandSolder, symbol Device:C
- removed D11: D_Schottky, Diode_SMD:D_SOD-123, symbol Device:D_Schottky
- removed D12: D, Diode_SMD:D_SMB, symbol Device:D
- removed F3: Polyfuse_Small, Resistor_SMD:R_1210_3225Metric, symbol Device:Polyfuse_Small
- removed J5: QR_connector, Connector_PinHeader_2.54mm:PinHeader_1x04_P2.54mm_Vertical, symbol Connector_Generic:Conn_01x04
- removed JP5, JP6: SolderJumper_2_Open, Jumper:SolderJumper-2_P1.3mm_Open_TrianglePad1.0x1.5mm, symbol Jumper:SolderJumper_2_Open
- removed R26, R27: 18k, Resistor_SMD:R_0603_1608Metric_Pad0.98x0.95mm_HandSolder, symbol Device:R
- removed R28: 1k, Resistor_SMD:R_0603_1608Metric_Pad0.98x0.95mm_HandSolder, symbol Device:R
- removed R29, R30: 10k, Resistor_SMD:R_0603_1608Metric_Pad0.98x0.95mm_HandSolder, symbol Device:R
- removed U9: PCF8523T, Package_SO:SOIC-8_3.9x4.9mm_P1.27mm, symbol Timer_RTC:PCF8523T
- removed Y2: 32768 Hz, Crystal:Crystal_SMD_EuroQuartz_EQ161-2Pin_3.2x1.5mm_HandSoldering, symbol Device:Crystal
- added LOGO3: Logo, sft:süff_10mm, symbol sft:Logo
Connections:
- net V3P3: now also U7.12 (AVREF), U7.13 (BVREF)
Other:
- note removed: "RTC"
- note removed: "TODO: define ratio!!"
- moved on the sheet: C27, C3, J4, M1, U1
